File: kicad/esp8266_irrigation_system.kicad_pcb (KiCad board)
At the start: 2 copper layers, 27 parts, among them J1 MOIST_CONN, P1 12V_POWER, P2 Serial, P3 DHT22_CONN, Q1 IRF540N, SW1 SW_PUSH, U1 MIC39100-3.3WS, U2 ESP8266-12F, U3 LM7805CT

Commit message: board re-done for fabrication
Parts:
- removed C1: 10uF, Capacitors_ThroughHole:CP_Radial_D5.0mm_P2.50mm
- removed C3: 1uF, Capacitors_ThroughHole:CP_Radial_D5.0mm_P2.50mm
- removed C4: 100n, Capacitors_ThroughHole:C_Disc_D3.8mm_W2.6mm_P2.50mm
- removed the REF** at (162.4, 62.2)
- removed the REF** at (111.3, 133.3)
- removed the REF** at (162.4, 133.3)
- removed the REF** at (111.3, 62.2)
- removed U1: MIC39100-3.3WS, TO_SOT_Packages_SMD:SOT-223
- removed U3: LM7805CT, TO_SOT_Packages_THT:TO-220_Vertical
- added J2: AUX_PINS, Pin_Headers:Pin_Header_Straight_2x03_Pitch2.54mm, F.Cu at (127.1, 99.9)
- added R3: 100R, Resistors_ThroughHole:R_Axial_DIN0207_L6.3mm_D2.5mm_P10.16mm_Horizontal, F.Cu at (117.7, 82.8)
- added R8: 10k, Resistors_SMD:R_1206_HandSoldering, F.Cu at (119.8, 86.3)
- added R9: 10k, Resistors_SMD:R_1206_HandSoldering, F.Cu at (154.3, 94.5)
- added REF**: Via-0.6mm, More:Via-0.6mm, F.Cu at (130.5, 77.6)
- added REF**: Via-0.6mm, More:Via-0.6mm, F.Cu at (141.1, 82.9)
- added REF**: Via-0.6mm, More:Via-0.6mm, F.Cu at (139.9, 82.9)
- added REF**: Via-0.6mm, More:Via-0.6mm, F.Cu at (141.1, 81.7)
- added REF**: Via-0.6mm, More:Via-0.6mm, F.Cu at (139.9, 81.7)
- added REF**: Via-0.6mm, More:Via-0.6mm, F.Cu at (141.1, 80.5)
- added REF**: Via-0.6mm, More:Via-0.6mm, F.Cu at (161.6, 103.7)
- added REF**: Via-0.6mm, More:Via-0.6mm, F.Cu at (160.4, 103.7)
- added REF**: Via-0.6mm, More:Via-0.6mm, F.Cu at (159.2, 103.7)
- added REF**: Via-0.6mm, More:Via-0.6mm, F.Cu at (161.6, 102.5)
- added REF**: Via-0.6mm, More:Via-0.6mm, F.Cu at (160.4, 102.5)
- added REF**: Via-0.6mm, More:Via-0.6mm, F.Cu at (129.3, 77.6)
- added REF**: Via-0.6mm, More:Via-0.6mm, F.Cu at (159.2, 102.5)
- added REF**: Via-0.6mm, More:Via-0.6mm, F.Cu at (161.6, 101.3)
- added REF**: Via-0.6mm, More:Via-0.6mm, F.Cu at (160.4, 101.3)
- added REF**: Via-0.6mm, More:Via-0.6mm, F.Cu at (159.2, 101.3)
- added REF**: Via-0.6mm, More:Via-0.6mm, F.Cu at (161.6, 100.1)
- added REF**: Via-0.6mm, More:Via-0.6mm, F.Cu at (160.4, 100.1)
- added REF**: MountingHole_3.2mm_M3, Mounting_Holes:MountingHole_3.2mm_M3, F.Cu at (157.5, 61.7)
- added REF**: MountingHole_3.2mm_M3, Mounting_Holes:MountingHole_3.2mm_M3, F.Cu at (118.9, 102.4)
- added REF**: Via-0.6mm, More:Via-0.6mm, F.Cu at (159.2, 100.1)
- added REF**: Via-0.6mm, More:Via-0.6mm, F.Cu at (139.9, 80.5)
- added REF**: Via-0.6mm, More:Via-0.6mm, F.Cu at (128.1, 77.6)
- added REF**: Via-0.6mm, More:Via-0.6mm, F.Cu at (126.9, 76.4)
- added REF**: Via-0.6mm, More:Via-0.6mm, F.Cu at (126.9, 77.6)
- added REF**: Via-0.6mm, More:Via-0.6mm, F.Cu at (130.5, 76.4)
- added REF**: Via-0.6mm, More:Via-0.6mm, F.Cu at (129.3, 76.4)
- added REF**: Via-0.6mm, More:Via-0.6mm, F.Cu at (128.1, 76.4)
- added REF**: Via-0.6mm, More:Via-0.6mm, F.Cu at (141.1, 84.1)
- added REF**: Via-0.6mm, More:Via-0.6mm, F.Cu at (139.9, 84.1)
- C2: footprint Capacitors_ThroughHole:C_Disc_D3.8mm_W2.6mm_P2.50mm -> Capacitors_SMD:C_1206_HandSoldering
- D1: value LED -> ACT-LED
- D2: value LED -> PWRLED
- J1: value MOIST_CONN -> 3V3_POWER; footprint Pin_Headers:Pin_Header_Straight_1x03_Pitch2.54mm -> Connect:bornier2
- L1: value INDUCTOR -> VALVE
- Q1: value IRF540N -> IRLL024NPBF; footprint Power_Integrations:TO-220 -> TO_SOT_Packages_SMD:SOT-223-3Lead_TabPin2
- R2, R4, R5, R6, R7, U2: moved to F.Cu
- SW1: value SW_PUSH -> RESET_SW
- moved P3 41.7 mm to (154.4, 78.2), turned to 90 degrees
- moved R6 35.6 mm to (154.3, 101.5), turned to 90 degrees
- moved J1 33.8 mm to (148.7, 62.6), turned to 180 degrees
- moved SW1 31.7 mm to (127.1, 90.3), turned to 270 degrees
- moved P2 30.1 mm to (160.7, 69.3)
- moved R4 23.7 mm to (149.1, 72.1), turned to 180 degrees
- moved R7 19.8 mm to (157.4, 94.5), turned to 90 degrees
- moved R5 18.8 mm to (140.2, 72.1)
- moved C2 17.1 mm to (128.5, 103.5), turned to 180 degrees
- moved U2 14.6 mm to (143.1, 86.5), turned to 0 degrees
- moved R2 14.2 mm to (131.4, 70.3), turned to 90 degrees
- moved P1 13.4 mm to (137.0, 62.6), turned to 180 degrees
- moved R1 10.5 mm to (143.9, 103.1)
- moved D2 10.2 mm to (134.7, 68.8), turned to 0 degrees
- moved D1 8.52 mm to (149.9, 103.1), turned to 270 degrees
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Connections:
- J1 pad 1: 5V -> 3.3V
- J1 pad 2: MOISTURE_SENSOR -> GND
- P2 pad 3: (no net) -> 3.3V
- Q1 pad 1: WATER_VALVE -> Net-(Q1-Pad1)
- U2 pad 17: (no net) -> Net-(R9-Pad2)
- U2 pad 2: (no net) -> ADC
- U2 pad 20: (no net) -> GPIO5
- U2 pad 4: (no net) -> GPIO16
- U2 pad 7: MOISTURE_SENSOR -> GPIO13
Routing:
- net 12V: track 64.0 -> 20.7 mm
- net MOISTURE_SENSOR: track 43.1 -> 0.00 mm, vias 2 -> 0
- net WATER_VALVE: track 51.2 -> 11.8 mm, vias 2 -> 1
- net GPIO5: track 0.00 -> 31.2 mm, vias 0 -> 2
- net 5V: track 30.1 -> 0.00 mm
- net ADC: track 0.00 -> 18.7 mm
- net GPIO13: track 0.00 -> 14.6 mm
- net INFO_LED: track 2.75 -> 14.9 mm, vias 0 -> 1
- net GPIO16: track 0.00 -> 11.2 mm
- net Net-(Q1-Pad1): track 0.00 -> 7.00 mm
- net Net-(D3-Pad2): track 25.5 -> 18.8 mm
- net GND: track 0.00 -> 6.60 mm
- net DHT22: track 9.67 -> 14.3 mm
- net Net-(R9-Pad2): track 0.00 -> 3.45 mm
- net DTR: track 32.6 -> 29.3 mm
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Other:
- board outline added: 48.6 x 50 mm
- board text added: "ADC"
- board text added: "DATA"
- board text added: "DTR"
- board text added: "GND"
- board text added: "GPIO13"
- board text added: "GPIO16"
- board text added: "GPIO5"
- board text added: "RST"
- board text added: "RX"
- board text added: "TX"
- board text added: "VCC"
