File: kicad/esp8266_irrigation_system.sch (KiCad schematic (older format))
At the start: 23 parts, among them J1 MOIST_CONN, P1 12V_POWER, P2 Serial, P3 DHT22_CONN, Q1 IRF540N, SW1 SW_PUSH, U1 MIC39100-3.3WS, U2 ESP8266-12F, U3 LM7805CT

Commit message: board re-done for fabrication
Parts:
- removed C1: 10uF, Capacitors_ThroughHole:CP_Radial_D5.0mm_P2.50mm, symbol C
- removed C3: 1uF, Capacitors_ThroughHole:CP_Radial_D5.0mm_P2.50mm, symbol C
- removed C4: 100n, Capacitors_ThroughHole:C_Disc_D3.8mm_W2.6mm_P2.50mm, symbol C
- removed J1: MOIST_CONN, Pin_Headers:Pin_Header_Straight_1x03_Pitch2.54mm, symbol CONN_01X03
- removed U1: MIC39100-3.3WS, TO_SOT_Packages_SMD:SOT-223, symbol MIC39100-3.3WS
- removed U3: LM7805CT, TO_SOT_Packages_THT:TO-220_Vertical, symbol LM7805CT
- added J1: 3V3_POWER, Connect:bornier2, symbol CONN_01X02
- added J2: AUX_PINS, Pin_Headers:Pin_Header_Straight_2x03_Pitch2.54mm, symbol CONN_02X03
- added R3: 100R, Resistors_ThroughHole:R_Axial_DIN0207_L6.3mm_D2.5mm_P10.16mm_Horizontal, symbol R
- added R8, R9: 10k, Resistors_SMD:R_1206_HandSoldering, symbol R
- C2: footprint Capacitors_ThroughHole:C_Disc_D3.8mm_W2.6mm_P2.50mm -> Capacitors_SMD:C_1206_HandSoldering
- Q1: footprint Power_Integrations:TO-220 -> TO_SOT_Packages_SMD:SOT-223-3Lead_TabPin2
Connections:
- net 3.3V: now also P2.3 (P3), J1.1 (P1), J2.1 (P1), R9.1
- net GND: now also J1.2 (P2), J2.6 (P6), R8.2
- net WATER_VALVE: now also R3.2; no longer Q1.1 (G)
- net at U2.17 (GPIO02): now also R9.2
- net ADC: now reaches U2.2 (ADC)
- net ADC: now also J2.4 (P4)
- net GPIO5: now reaches U2.20 (GPIO05)
- net GPIO5: now also J2.3 (P3)
- net GPIO16: now reaches U2.4 (GPIO16)
- net GPIO16: now also J2.5 (P5)
- net MOISTURE_SENSOR renamed GPIO13
- net GPIO13: now also J2.2 (P2)
- new net: Q1.1 (G), R3.1, R8.1
- no-connect marks 11 -> 6
Other:
- moved on the sheet: R6
